File: boards/XR-VCO-core/XR-VCO-core.sch (KiCad schematic (older format))
At the start: 64 parts, among them J1 Conn_01x08_Male, J2 Conn_01x08_Male, J3 Conn_02x08_Odd_Even, Q1 2N3404, Q2 LM394, SW1 SW_DPDT_x2, U1 TL074, U2 XR2206, U3 TL074

Commit message: Reshuffling and adding docs
Parts:
- U1: renamed from U3; footprint Housings_DIP:DIP-14_W7.62mm_Socket_LongPads -> Housings_DIP:DIP-14_W7.62mm_LongPads
- U2: renamed from U1; value TL074 -> TL072; symbol TL074 -> TL072
- renumbered U2 to U3
Connections:
- net +12V: now also U2.8 (V+), U2.8 (V+); no longer U2.4 (V+), U2.4 (V+)
- net -12VA: now also U2.4 (V-), U2.4 (V-); no longer U2.11 (V-), U2.11 (V-)
- net Earth: now also U1.12 (+), U1.3 (+), U1.5 (+), U2.5 (+); no longer U1.12 (+), U1.5 (+), U1.5 (+), U2.10 (+)
- net SkewCV: no longer D5.2 (A), D6.1 (K), R25.2, U3.1 (AMSI)
- net at D2.1 (K), R13.2, R5.1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: now also U1.2 (-); no longer U1.6 (-)
- net at D3.1 (K): now also U1.1; no longer U1.7
- net at R16.1, R17.2: now also U1.6 (-); no longer U1.13 (-)
- net at D5.1 (K), R17.1: now also U1.7; no longer U1.14
- net at C3.2, Q2.6 (C1), R11.1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: now also U2.6 (-); no longer U2.9 (-)
- net at C3.1, R14.2, RV4.2: now also U2.7; no longer U2.8
- net at R24.1, R26.1: now also U1.9 (-); no longer U1.2 (-)
- net at R26.2, R28.1: now also U1.8; no longer U1.1
- net at R21.1, R22.2: now also U1.10 (+); no longer U1.3 (+)
- net at R27.2, R33.1, RV7.1: now also U1.13 (-); no longer U1.6 (-)
- net at R33.2, R36.1: now also U1.14; no longer U1.7
- new net Skew: D5.2 (A), D6.1 (K), R25.2, U3.1 (AMSI)
